Commit message: Scaled down dimensions of mesh in URDF file

File: software/ros_packages/mr1819-arm_urdf/urdf/mr1819-arm_urdf.urdf (robot description, URDF)
Before this commit: robot mr1819-arm_urdf, 7 links, 6 joints
Links:
- link base_link: geometry collision mesh filename=package://mr1819-arm_urdf/meshes/base_link.STL scale=0.001 0.001 0.001; visual mesh filename=package://mr1819-arm_urdf/meshes/base_link.STL scale=0.001 0.001 0.001
- link elbow_roll: geometry collision mesh filename=package://mr1819-arm_urdf/meshes/elbow_roll.STL scale=0.001 0.001 0.001; visual mesh filename=package://mr1819-arm_urdf/meshes/elbow_roll.STL scale=0.001 0.001 0.001
- link gripper: geometry collision mesh filename=package://mr1819-arm_urdf/meshes/gripper.STL scale=0.001 0.001 0.001; visual mesh filename=package://mr1819-arm_urdf/meshes/gripper.STL scale=0.001 0.001 0.001
- link shoulder: geometry collision mesh filename=package://mr1819-arm_urdf/meshes/shoulder.STL scale=0.001 0.001 0.001; visual mesh filename=package://mr1819-arm_urdf/meshes/shoulder.STL scale=0.001 0.001 0.001
- link upper_arm: geometry collision mesh filename=package://mr1819-arm_urdf/meshes/upper_arm.STL scale=0.001 0.001 0.001; visual mesh filename=package://mr1819-arm_urdf/meshes/upper_arm.STL scale=0.001 0.001 0.001
- link wrist_pitch: geometry collision mesh filename=package://mr1819-arm_urdf/meshes/wrist_pitch.STL scale=0.001 0.001 0.001; visual mesh filename=package://mr1819-arm_urdf/meshes/wrist_pitch.STL scale=0.001 0.001 0.001
- link wrist_roll: geometry collision mesh filename=package://mr1819-arm_urdf/meshes/wrist_roll.STL scale=0.001 0.001 0.001; visual mesh filename=package://mr1819-arm_urdf/meshes/wrist_roll.STL scale=0.001 0.001 0.001
