Commit message: Make arm fixed in Gazebo

File: software/ros_packages/mr1920_arm_urdf_export/urdf/mr1920_arm_urdf_export.urdf (robot description, URDF)
Before this commit: robot mr1920_arm_urdf_export, 7 links, 6 joints
Links:
- added link world
Joints:
- added joint base_fixed: type fixed, parent world, child base_link, origin xyz=0 0 0 rpy=0 0 0
