Commit message: Change shoulder pitch limits

File: software/ros_packages/rover_arm_description/urdf/mr1920_arm_urdf_export.urdf (robot description, URDF)
Before this commit: robot mr1920_arm_urdf_export, 8 links, 7 joints
Joints:
- joint shoulder_pitch: limit lower=-6.28 upper=6.28 effort=150.0 velocity=3.15 -> lower=-1.57 upper=1.57 effort=150.0 velocity=3.15

Commit message: Tighten joint limits

File: software/ros_packages/rover_arm_description/urdf/mr1920_arm_urdf_export.urdf (robot description, URDF)
Before this commit: robot mr1920_arm_urdf_export, 8 links, 7 joints
Joints:
- joint base_roll: limit lower=-6.28 upper=6.28 effort=150.0 velocity=3.15 -> lower=-3.14 upper=3.14 effort=150.0 velocity=3.15
- joint elbow_pitch: limit lower=-6.28 upper=6.28 effort=150.0 velocity=3.15 -> lower=-3.14 upper=3.14 effort=150.0 velocity=3.15
- joint elbow_roll: limit lower=-6.28 upper=6.28 effort=150.0 velocity=3.15 -> lower=-3.14 upper=3.14 effort=150.0 velocity=3.15
- joint wrist_pitch: limit lower=-6.28 upper=6.28 effort=150.0 velocity=3.15 -> lower=-3.14 upper=3.14 effort=150.0 velocity=3.15
