Commit message: Update starting configuration

File: software/ros_packages/rover_arm_ik/rover_arm_description/urdf/mr1920_arm_urdf_export.urdf (robot description, URDF)
Before this commit: robot mr1920_arm_urdf_export, 8 links, 7 joints
Joints:
- joint base_roll: origin xyz=0.14566 -0.14314 0.11421 rpy=1.5708 0 -0.11656 -> xyz=0.14566 -0.14314 0.11421 rpy=1.5708 0 0
- joint elbow_pitch: origin xyz=0 0 0.52362 rpy=1.4974 0 0 -> xyz=0 0 0.52362 rpy=0 0 0
- joint elbow_roll: origin xyz=-0.01623 0 0.035461 rpy=0 0 0.0027091 -> xyz=-0.01623 0 0.035461 rpy=0 0 3.1416
- joint shoulder_pitch: origin xyz=0.017768 0.082744 0 rpy=-1.7023 0 0 -> xyz=0.017768 0.082744 0 rpy=-1.5708 0 0
- joint wrist_pitch: origin xyz=0.052628 0 0.35621 rpy=-0.11133 0 3.1416 -> xyz=0.052628 0 0.35621 rpy=0 0 3.1416
- joint wrist_roll: origin xyz=-0.069133 0 0.053575 rpy=1.5708 0 -2.9823 -> xyz=-0.069133 0 0.053575 rpy=1.5708 0 -1.5708

Commit message: Update arm limits

File: software/ros_packages/rover_arm_ik/rover_arm_description/urdf/mr1920_arm_urdf_export.urdf (robot description, URDF)
Before this commit: robot mr1920_arm_urdf_export, 8 links, 7 joints
Joints:
- joint base_roll: limit lower=-3.14 upper=3.14 effort=150.0 velocity=3.15 -> lower=-0.7854 upper=0.7854 effort=150.0 velocity=3.15
- joint elbow_pitch: limit lower=-3.14 upper=3.14 effort=150.0 velocity=3.15 -> lower=-1.5708 upper=1.5708 effort=150.0 velocity=3.15
- joint elbow_roll: limit lower=-3.14 upper=3.14 effort=150.0 velocity=3.15 -> lower=-1.5708 upper=1.5708 effort=150.0 velocity=3.15
- joint shoulder_pitch: limit lower=-1.57 upper=1.57 effort=150.0 velocity=3.15 -> lower=-1.5708 upper=1.5708 effort=150.0 velocity=3.15
- joint wrist_pitch: limit lower=-3.14 upper=3.14 effort=150.0 velocity=3.15 -> lower=-1.5708 upper=1.5708 effort=150.0 velocity=3.15
- joint wrist_roll: limit lower=-6.28 upper=6.28 effort=150.0 velocity=3.15 -> (none); type revolute -> continuous
